Commit message: Moved all seperate parts to origin in Onshape and reimported and tuned

File: arctos_defs/arctos.urdf (robot description, URDF)
Before this commit: robot onshape, 9 links, 8 joints
Links:
- link arctos_base: mass 1.0413378737551433062 -> 1.041338
- link arctos_lower: mass 1.4118318629235360184 -> 1.411832
- link arctos_middle: mass 1.5722421951083009883 -> 1.572243
- link arctos_upper: mass 0.6272436456112834291 -> 0.627244
- link gripper_assembly_inner: mass 0.19463214953987617584 -> 0.194632
- link gripper_assembly_outer: mass 0.13208625646334956616 -> 0.133828
- link left_jaw: mass 0.0104625931880081742 -> 0.010463
- link right_jaw: mass 0.010168042155151081618 -> 0.010168
- link wrist: mass 0.56700886652075166428 -> 0.567009
Joints:
- joint inner_wrist: limit lower=-1.6580627893946131568 upper=1.6580627893946131568 effort=12 velocity=20 -> lower=-1.74533 upper=1.74533 effort=70 velocity=20; origin xyz=0.00021854809329471813761 0.0017743655747750608498 -0.12542436358686440134 rpy=-6.9874661612348195789e-15 1.5707963267948850117 0 -> xyz=0.000219 0.001774 -0.125424 rpy=0 1.5708 0
- joint lower_base: limit lower=-6.283185307179586232 upper=6.283185307179586232 effort=12 velocity=20 -> lower=-4.71239 upper=4.71239 effort=70 velocity=20; origin xyz=-0.00052900000000000169109 0 0.12990600176195876703 rpy=-3.1415926535897926719 2.4377752293772548502e-17 1.4977683394279026321e-14 -> xyz=-0.000529 0 0.129906 rpy=-3.14159 0 0.004351
- joint middle_lower: limit lower=-1.3089969389957472057 upper=2.356194490192344837 effort=12 velocity=20 -> lower=-1.22173 upper=2.18166 effort=70 velocity=20; origin xyz=0.020885040968205974277 0.00086987140237410553144 -0.15772234492155495778 rpy=1.5707963267950006969 -0.06504782007281141587 1.5951947608009762544e-16 -> xyz=0.020885 0.000870 -0.157722 rpy=1.5708 0 0
- joint outer_inner: limit lower=-3.4906585039886590671 upper=3.4906585039886590671 effort=12 velocity=20 -> lower=-4.71239 upper=4.71239 effort=70 velocity=20; origin xyz=0.039835445112786860289 -2.2204460492503130808e-15 -3.6776137690708310402e-15 rpy=-1.5707963267949791586 1.3778210289552164092 1.5707963267947004926 -> xyz=0.039835 0 0 rpy=1.5708 0 -1.5708
- joint slide_left: limit lower=-0.015 upper=0.0 effort=12 velocity=20 -> lower=-0.015 upper=0 effort=70 velocity=20; origin xyz=-0.012068082601611365701 -0.029103138881718670916 -0.040243588945377273269 rpy=1.5707963267948992225 1.5707963267948146235 0 -> xyz=0.007431 0.030780 -0.040326 rpy=-1.5708 1.5708 0
- joint slide_right: limit lower=0.0 upper=0.015 effort=12 velocity=20 -> lower=-0.015 upper=0 effort=70 velocity=20; mimic joint=slide_left -> joint=slide_left multiplier=-1 offset=0; origin xyz=0.0074314381148364444529 0.015896861565316222631 -0.040325652756017238421 rpy=-1.5707963267948970021 1.5707963267948092945 0 -> xyz=-0.012068 -0.028986 -0.040244 rpy=1.5708 1.5708 0
- joint upper_middle: limit lower=-1.8325957145940461324 upper=0.87266462599716476678 effort=12 velocity=20 -> lower=-1.91986 upper=0.87266 effort=70 velocity=20; origin xyz=-0.0013103630346719770308 -0.26100665594985539286 0.0054290868549383020786 rpy=-1.0765344187740975265e-13 8.1164530008389699728e-15 0.0040744247603443310007 -> xyz=-0.001310 -0.261007 0.005429 rpy=0 0 0
- joint wrist_upper: limit lower=-3.2288591161895094928 upper=3.2288591161895094928 effort=12 velocity=20 -> lower=-4.71239 upper=4.71239 effort=70 velocity=20; origin xyz=0.13874345514589062067 -0.021748655380295134343 -0.0054925270810687130268 rpy=-1.5707963267948807928 -1.5245022596773765144 1.5688068046258516475 -> xyz=0.138743 -0.021749 -0.005493 rpy=-0.001990 -1.5708 0
